Commit message: some changes

File: urdf/sensors/kinetic_rgb.urdf.xacro (robot description, xacro)
@@ -2,4 +2,5 @@
 <robot xmlns:xacro="http://ros.org/wiki/xacro">
   <xacro:include filename="$(find cobot_simulation)/urdf/sensors/kinetic_rgb.gazebo.xacro"/>
+  <!-- if not defined, camera doesn't spawn -->
   <xacro:macro name="dummy_inertial">
         <inertial>
@@ -28,7 +29,5 @@
             <visual>
                 <geometry>
-                <!--
-                <box size="0.06 0.1 0.03" />
-                    -->
+                <!-- <box size="0.06 0.1 0.03" /> -->
                             <mesh filename="package://cobot_simulation/meshes/sensors/camera/kinetic.stl"/>
                 </geometry>
